File: Hardware/Power_Board/Power_Board.sch (EAGLE design)
At the start: 28 parts, among them J1 BATTERY_CONNDEANS, Q1 MOSFET-PCHANNELFQP27P06, U1 TL431PTH

Commit message: Changed MOSFET to FQP27P06.
Parts:
- Q1: PART_NAME NDP6020P -> FQP27P06
Changed lines of the file:
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@@
 <part name="U1" library="SparkFun-AnalogIC" deviceset="TL431" device="PTH"/>
 <part name="Q1" library="SparkFun-DiscreteSemi" deviceset="MOSFET-PCHANNEL" device="FQP27P06">
-<attribute name="PART_NAME" value="NDP6020P"/>
+<attribute name="PART_NAME" value="FQP27P06"/>
 </part>
 <part name="GND2" library="SparkFun-Aesthetics" deviceset="GND" device=""/>
